File: Electrical/Microcontroller boards/Microcontroller boards.kicad_pcb (KiCad board)
At the start: 2 copper layers, 44 x 49.8 mm, 15 parts, among them J1 S4B-PH-K-SLFSN, J10 Conn_01x10_Pin, J2 S4B-PH-K-SLFSN, J3 Conn_01x03_Pin, J4 Conn_01x03_Pin, J5 Conn_01x03_Pin, J6 Conn_01x03_Pin, J7 Conn_01x03_Pin, J8 Conn_01x03_Pin, U1 NodeMCU1.0(ESP-12E)

Commit message: Update Microcontroller boards.kicad_pcb
Parts:
- renumbered G*** to swab
Changed lines of the file:
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@@
 		(tags "connector Wuerth WR-WTB vertical")
 		(property "Reference" "J4"
-			(at 1.5 -2.5 360)
+			(at 1.5 -2.5 0)
 			(layer "F.SilkS")
 			(effects
@@
 		)
 		(property "Value" "Conn_01x03_Pin"
-			(at 1.5 3.4 360)
+			(at 1.5 3.4 0)
 			(layer "F.Fab")
 			(effects
@@
 		)
 		(fp_text user "${REFERENCE}"
-			(at 1.5 1.5 360)
+			(at 1.5 1.5 0)
 			(layer "F.Fab")
 			(effects
@@
 			)
 		)
-		(fp_text user "G"
-			(at -11.43 15.24 0)
+		(fp_text user "swab"
+			(at -11.0098 15.2258 0)
 			(layer "F.SilkS")
 			(effects
@@
 		(layer "F.Cu")
 		(at 117.039133 82.114134)
-		(property "Reference" "G***"
+		(property "Reference" "swab"
 			(at 0.8382 13.6144 0)
 			(layer "F.SilkS")
