File: Electrical/PowerBoard2/PowerBoard2/PowerBoard2.kicad_pcb (KiCad board)
At the start: 2 copper layers, 11 parts, among them J1 XT60PW-M, J2 XT60PW-M, J5 XT60PW-M, U1 LMZ22005TZ/NOPB, U2 INA226AIDGSR

Commit message: powerboard design
Routing:
- added copper zone on F.Cu, net +5V
Changed lines of the file:
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@@
 		)
 		(property "Value" "0.005 R"
-			(at 0 2.28 360)
+			(at 0 2.28 0)
 			(layer "F.Fab")
 			(effects
@@
 		)
 		(fp_text user "${REFERENCE}"
-			(at 0 0 360)
+			(at 0 0 0)
 			(layer "F.Fab")
 			(effects
@@
 		)
 		(property "Value" "25SEK120M"
-			(at 8.89 5.005 360)
+			(at 8.89 5.005 0)
 			(layer "F.Fab")
 			(effects
@@
 		)
 		(property "Footprint" "Libraries:25SEK120M"
-			(at 0 0 360)
+			(at 0 0 0)
 			(layer "F.Fab")
 			(hide yes)
@@
 		)
 		(property "Datasheet" ""
-			(at 0 0 360)
+			(at 0 0 0)
 			(layer "F.Fab")
 			(hide yes)
@@
 		)
 		(property "Description" ""
-			(at 0 0 360)
+			(at 0 0 0)
 			(layer "F.Fab")
 			(hide yes)
@@
 		)
 		(property "Value" "25SEK120M"
-			(at 8.89 5.005 360)
+			(at 8.89 5.005 0)
 			(layer "F.Fab")
 			(effects
@@
 		)
 		(property "Footprint" "Libraries:25SEK120M"
-			(at 0 0 360)
+			(at 0 0 0)
 			(layer "F.Fab")
 			(hide yes)
@@
 		)
 		(property "Datasheet" ""
-			(at 0 0 360)
+			(at 0 0 0)
 			(layer "F.Fab")
 			(hide yes)
@@
 		)
 		(property "Description" ""
-			(at 0 0 360)
+			(at 0 0 0)
 			(layer "F.Fab")
 			(hide yes)
@@
 	)
 	(gr_line
-		(start 253.45 94.1)
-		(end 168.55 94.1)
+		(start 252.95 94.1)
+		(end 168.05 94.1)
 		(stroke
 			(width 0.1)
@@
 		(net 7)
 	)
+	(zone
+		(net 6)
+		(net_name "+5V")
+		(layer "F.Cu")
+		(hatch edge 0.5)
+		(connect_pads yes
+			(clearance 0)
+		)
+		(min_thickness 0.25)
+		(filled_areas_thickness no)
+		(fill yes
+			(thermal_gap 0.5)
+			(thermal_bridge_width 0.5)
+		)
+		(polygon
+			(pts
+				(xy 202 90.5) (xy 204.5 90.5) (xy 208 87) (xy 208 76) (xy 209.5 74.5) (xy 210.5 74.5) (xy 210.5 71.5)
+				(xy 208.876567 70.123433) (xy 208.348002 69.5) (xy 208.348002 69) (xy 208.348002 68.150801) (xy 206.849199 68.150801)
+				(xy 204.5 70.5) (xy 204.5 78) (xy 202 80.5)
+			)
+		)
+	)
+	(zone
+		(net 6)
+		(net_name "+5V")
+		(layer "F.Cu")
+		(hatch edge 0.5)
+		(priority 1)
+		(connect_pads yes
+			(clearance 0)
+		)
+		(min_thickness 0.25)
+		(filled_areas_thickness no)
+		(fill yes
+			(thermal_gap 0.5)
+			(thermal_bridge_width 0.5)
+		)
+		(polygon
+			(pts
+				(xy 204.5 90.5) (xy 205.5 91.5) (xy 224 91.5) (xy 225.5 90.5) (xy 225.5 88) (xy 224 87) (xy 208 87)
+			)
+		)
+	)
 )

Commit message: PowerBoard 2 first iteration
Parts:
- added C2: 300uF, Capacitor_SMD:C_0805_2012Metric_Pad1.18x1.45mm_HandSolder, F.Cu at (191.5, 81.5)
- added J3: B4B-XH-A_LF__SN_, B4B-XH-A_LF__SN_:JST_B4B-XH-A_LF__SN_, F.Cu at (187.8, 91.0)
- added R3: 10k, Resistor_SMD:R_0805_2012Metric_Pad1.20x1.40mm_HandSolder, F.Cu at (193.5, 77.0)
- added R4: 10k, Resistor_SMD:R_0805_2012Metric_Pad1.20x1.40mm_HandSolder, F.Cu at (189.0, 77.0)
- added U3: USB-A-S-RA-TSMT, _Footprints:USB-A-S-RA-TSMT_ADM, F.Cu at (178.8, 82.3)
- moved J2 3.40 mm to (181.7, 70.9)
- moved ShuntResistor1 2.60 mm to (189.8, 63.7)
- moved U2 2.60 mm to (190.5, 69.5)
Connections:
- J2 pad 2: Net-(J2--) -> +12V
- ShuntResistor1 pad 2: Net-(J2--) -> +12V
- U2 pad 1: unconnected-(U2-A1-Pad1) -> GND
- U2 pad 10: Net-(J2--) -> +12V
- U2 pad 2: unconnected-(U2-A0-Pad2) -> GND
- U2 pad 4: unconnected-(U2-SDA-Pad4) -> /SDA
- U2 pad 5: unconnected-(U2-SCL-Pad5) -> /SCL
- U2 pad 6: Net-(J2--) -> Net-(U2-VS)
- U2 pad 8: +5V -> /Buck Converter/Vin (12V)
Routing:
- net Net-(U2-VS): track 0.00 -> 35.1 mm, vias 0 -> 2
- net /SCL: track 0.00 -> 25.2 mm, vias 0 -> 2
- net /SDA: track 0.00 -> 23.5 mm, vias 0 -> 2
- net Net-(J2--): track 8.34 -> 0.00 mm
- net GND: track 0.00 -> 4.71 mm, vias 60 -> 63
- net +12V: track 0.00 -> 4.55 mm
- added copper zone on F.Cu, net +12V
- added copper zone on F.Cu, net /Buck Converter/Vin (12V)
- added copper zone on B.Cu, net GND

Commit message: Updated Schematic, Rerouted Some Things
Parts:
- removed R3, R4: 10k, Resistor_SMD:R_0805_2012Metric_Pad1.20x1.40mm_HandSolder
- moved C2 8.96 mm to (182.6, 81.2)
Routing:
- net Net-(U2-VS): track 35.1 -> 26.2 mm, vias 2 -> 1
- net /SCL: track 25.2 -> 19.8 mm, vias 2 -> 1
- net GND: track 4.71 -> 0.00 mm, vias 63 -> 64
- net /SDA: track 23.5 -> 20.7 mm, vias 2 -> 1
