File: Electrical/PowerBoard2/PowerBoard2/PowerBoard2.kicad_sch (KiCad schematic)
At the start: 5 parts, among them J1 XT60PW-M, J2 XT60PW-M, J5 XT60PW-M, U2 INA226AIDGSR

Commit message: PowerBoard 2 first iteration
Parts:
- added C2: 300uF, Capacitor_SMD:C_0805_2012Metric_Pad1.18x1.45mm_HandSolder, symbol Device:C
- added J3: B4B-XH-A_LF__SN_, B4B-XH-A_LF__SN_:JST_B4B-XH-A_LF__SN_, symbol B4B-XH-A_LF__SN_:B4B-XH-A_LF__SN_
- added R3, R4: 10k, Resistor_SMD:R_0805_2012Metric_Pad1.20x1.40mm_HandSolder, symbol Device:R
- added U3: USB-A-S-RA-TSMT, USB-A-S-RA-TSMT_ADM, symbol 2025-02-23_03-18-15:USB-A-S-RA-TSMT
Connections:
- net +5V: now also C2.1, U3.1; no longer U2.8 (VBUS)
- net Buck Converter/Vin (12V): now also U2.8 (VBUS)
- net GND: now also U2.1 (A1), U2.2 (A0), C2.2, J3.4, U3.4
- net SCL: now also J3.3, R3.1, R3.2
- net SDA: now also J3.2, R4.1, R4.2
- net +12V: now reaches J2.2 (-), ShuntResistor1.2, U2.10 (IN+)
- net +12V: no longer U2.6 (VS)
- new net: J3.1, U2.6 (VS)
Other:
- moved on the sheet: J1, J2, ShuntResistor1

Commit message: Updated Schematic, Rerouted Some Things
Parts:
- removed R3, R4: 10k, Resistor_SMD:R_0805_2012Metric_Pad1.20x1.40mm_HandSolder, symbol Device:R
Connections:
- no-connect marks 0 -> 3
Other:
- moved on the sheet: C2, J5, U3
